File: rcbus-ymf262.kicad_sch (KiCad schematic)
At the start: 41 parts, among them CON1 SJ1-3523N, P1 RC2014 BUS, U1 74HCT688, U2 YMF262, U3 YAC512, U4 TL074, Y1 SG-8002CA

Commit message: reorg
Connections:
- net AUDIO_CH1: now also C9.1, U4.10 (+); no longer C10.1, U4.12 (+)
- net AUDIO_CH2: now also C10.1, U4.12 (+); no longer C9.1, U4.10 (+)
- net L: now also C14.2, R9.2, U4.14; no longer C13.1, R8.2, U4.8
- net R: now also C13.1, R8.2, U4.8; no longer C14.2, R9.2, U4.14
Other:
- moved on the sheet: C10, C13, C14, C9, R8, R9, U4C, U4D
